File: hardware/bison_module/bison_module.kicad_pcb (KiCad board)
At the start: 2 copper layers, 39 parts, among them J1 Conn_01x02, J2 Conn_01x02, J3 Conn_01x04, J4 Conn_01x02, J5 Conn_01x03, J6 Conn_01x02, J7 Conn_01x02, Q1 AO3401A, Q2 AO3401A, U1 ESP-12E, U2 LM1117-3.3, U3 TB6612FNG, U4 TB6612FNG

Commit message: more pcb layout
Parts:
- removed the J2 at (164.6, 131.2)
- removed Q2: AO3401A, Package_TO_SOT_SMD:SOT-23
- removed the R1 at (183.4, 126.2)
- removed the R6 at (189.2, 118.0)
- added C2: 4.7uF, Capacitor_Tantalum_SMD:CP_EIA-3216-18_Kemet-A, B.Cu at (135.0, 99.5)
- added C4: 100nF, Capacitor_SMD:C_0805_2012Metric, F.Cu at (125.5, 96.5)
- added C5: 100nF, Capacitor_SMD:C_0805_2012Metric, F.Cu at (110.5, 86.5)
- added D2: D, Diode_SMD:D_0805_2012Metric, B.Cu at (136.3, 88.2)
- added R4: 10k, Resistor_SMD:R_0805_2012Metric, B.Cu at (108.5, 95.5)
- added R5: 10k, Resistor_SMD:R_0805_2012Metric, F.Cu at (108.0, 86.5)
- added R9: 10k, Resistor_SMD:R_0805_2012Metric, B.Cu at (108.5, 98.0)
- added SW1: SW_SPST, Connector_AMASS:AMASS_XT30U-F_1x02_P5.0mm_Vertical, F.Cu at (106.0, 114.5)
- added SW2: SW_Push, Button_Switch_SMD:SW_Push_1P1T_NO_6x6mm_H9.5mm, F.Cu at (123.0, 89.5)
- added SW3: SW_Push, Button_Switch_SMD:SW_Push_1P1T_NO_6x6mm_H9.5mm, F.Cu at (115.5, 89.5)
- C1: renamed from C2; moved to B.Cu
- C10: renamed from C7; moved to B.Cu
- C11: renamed from C8; moved to B.Cu
- C3: renamed from C1; footprint Capacitor_THT:CP_Radial_D10.0mm_P5.00mm -> Capacitor_THT:CP_Radial_D10.0mm_P7.50mm
- C6: renamed from C3; moved to B.Cu
- C7: renamed from C4; moved to B.Cu
- D1, R7, R8, U1: moved to B.Cu
- D3: renamed from D2; moved to B.Cu
- D4: renamed from D3; value BLUE -> B; moved to B.Cu
- D5: renamed from D4; value YELLOW -> Y; moved to B.Cu
- D6: renamed from D5; value GREEN -> G; moved to B.Cu
- Q1: value AO3401A -> QM6015D; footprint Package_TO_SOT_SMD:SOT-23 -> Package_TO_SOT_SMD:TO-252-2
- R1: renamed from R2; moved to B.Cu
- R10: renamed from R9; moved to B.Cu
- R11: renamed from R10; moved to B.Cu
- R12: renamed from R11; moved to B.Cu
- R13: renamed from R12; moved to B.Cu
- R14: renamed from R13; moved to B.Cu
- R3: renamed from R4; moved to B.Cu
- R6: renamed from R5; moved to B.Cu
- moved J4 77.2 mm to (104.5, 98.0)
- moved R10 72.0 mm to (121.8, 115.0), turned to 180 degrees
- moved D3 70.6 mm to (108.5, 104.0)
- moved R11 70.3 mm to (108.4, 101.2)
- moved D6 63.3 mm to (123.0, 104.5), turned to 90 degrees
- moved R2 62.8 mm to (123.0, 96.5), turned to 90 degrees
- moved C9 62.2 mm to (111.0, 100.5), turned to 90 degrees
- moved R6 61.0 mm to (128.2, 116.2), turned to 180 degrees
- moved R1 59.1 mm to (117.5, 115.0)
- moved R3 58.5 mm to (136.4, 86.0), turned to 180 degrees
- moved C1 56.8 mm to (134.5, 97.0)
- moved R12 56.4 mm to (130.0, 108.5), turned to -90 degrees
- moved R13 56.3 mm to (126.5, 108.4), turned to -90 degrees
- moved D4 55.3 mm to (130.0, 104.6), turned to 90 degrees
- moved U4 54.8 mm to (133.0, 89.5), turned to 180 degrees
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- renumbered C5 to C8, C6 to C9, J3 to J2, J4 to J3, J5 to J4, J6 to J5, J7 to J6, R3 to R2
Connections:
- J2 pad 1: +3V3 -> ESP_TX
- J2 pad 3: ESP_TX -> GND
- J2 pad 4: GND -> +3V3
- Q1 pad 2: Net-(J1-Pad1) -> V_POWER
- R1 pad 2: Net-(Q2-Pad1) -> Net-(Q1-Pad1)
- R2 pad 2: Net-(R3-Pad2) -> Net-(C4-Pad1)
- R3 pad 2: Net-(R4-Pad2) -> Net-(R3-Pad2)
- R7 pad 1: Net-(Q2-Pad1) -> Net-(Q1-Pad1)
- U1 pad 1: Net-(R4-Pad2) -> Net-(C4-Pad1)
- U1 pad 13: unconnected-(U1-Pad13) -> MOT_R_IN1
- U1 pad 14: unconnected-(U1-Pad14) -> MOT_R_IN2
- U1 pad 16: MOT_R_PWM -> Net-(R9-Pad1)
- U1 pad 17: MOT_R_IN1 -> Net-(R4-Pad2)
- U1 pad 18: MOT_R_IN2 -> Net-(C5-Pad1)
- U1 pad 4: unconnected-(U1-Pad4) -> MOT_L_IN1
- U1 pad 6: MOT_L_IN1 -> MOT_R_PWM
Other:
- board outline added: 40.5 x 33.5 mm
