File: hardware/bison_module/bison_module.kicad_sch (KiCad schematic)
At the start: 39 parts, among them J1 Conn_01x02, J2 Conn_01x02, J3 Conn_01x04, J4 Conn_01x02, J5 Conn_01x03, J6 Conn_01x02, J7 Conn_01x02, Q1 AO3401A, Q2 AO3401A, U1 ESP-12E, U2 LM1117-3.3, U3 TB6612FNG, U4 TB6612FNG

Commit message: ESP programming stuff
Parts:
- added C2: 4.7uF, Capacitor_Tantalum_SMD:CP_EIA-3216-18_Kemet-A, symbol Device:C_Polarized
- added C4, C5: 100nF, Capacitor_SMD:C_0805_2012Metric, symbol Device:C
- added D?: D, symbol Device:D_Schottky
- added R11, R5, R6: 10k, Resistor_SMD:R_0805_2012Metric, symbol Device:R
- added SW1: SW_Push, symbol Switch:SW_Push
- added SW2: SW_SPST, symbol Switch:SW_SPST
- C1: renamed from C2; footprint (none) -> Capacitor_SMD:C_0805_2012Metric
- C10: renamed from C7; footprint (none) -> Capacitor_SMD:C_0805_2012Metric
- C11: renamed from C8; footprint (none) -> Capacitor_SMD:C_0805_2012Metric
- C3: renamed from C1; footprint (none) -> Capacitor_THT:CP_Radial_D10.0mm_P5.00mm
- C6: renamed from C3; footprint (none) -> Capacitor_SMD:C_0805_2012Metric
- C7: renamed from C4; footprint (none) -> Capacitor_Tantalum_SMD:CP_EIA-3216-18_Kemet-A
- C8: renamed from C5; footprint (none) -> Capacitor_Tantalum_SMD:CP_EIA-3216-18_Kemet-A
- C9: renamed from C6; footprint (none) -> Capacitor_SMD:C_0805_2012Metric
- D1, D2: footprint (none) -> LED_SMD:LED_0805_2012Metric
- D3: value BLUE -> B; footprint (none) -> LED_SMD:LED_0805_2012Metric
- D4: value YELLOW -> Y; footprint (none) -> LED_SMD:LED_0805_2012Metric
- D5: value GREEN -> G; footprint (none) -> LED_SMD:LED_0805_2012Metric
- J1, J4: footprint (none) -> Connector_AMASS:AMASS_XT30U-F_1x02_P5.0mm_Vertical
- J2, J6, J7: footprint (none) -> Connector_PinHeader_2.54mm:PinHeader_1x02_P2.54mm_Vertical
- J3: footprint (none) -> Connector_PinHeader_2.54mm:PinHeader_1x04_P2.54mm_Vertical
- J5: footprint (none) -> Connector_PinHeader_2.54mm:PinHeader_1x03_P2.54mm_Vertical
- R1, R2, R3, R4: footprint (none) -> Resistor_SMD:R_0805_2012Metric
- R10: renamed from R8; footprint (none) -> Resistor_SMD:R_0805_2012Metric
- R12: renamed from R9; footprint (none) -> Resistor_SMD:R_0805_2012Metric
- R13: renamed from R10; footprint (none) -> Resistor_SMD:R_0805_2012Metric
- R14: renamed from R11; footprint (none) -> Resistor_SMD:R_0805_2012Metric
- R15: renamed from R12; footprint (none) -> Resistor_SMD:R_0805_2012Metric
- R16: renamed from R13; footprint (none) -> Resistor_SMD:R_0805_2012Metric
- R7: renamed from R5; footprint (none) -> Resistor_SMD:R_0805_2012Metric
- R8: renamed from R6; footprint (none) -> Resistor_SMD:R_0805_2012Metric
- R9: renamed from R7; footprint (none) -> Resistor_SMD:R_0805_2012Metric
- U2: footprint (none) -> Package_TO_SOT_SMD:SOT-223-3_TabPin2
Connections:
- net +3V3: now also J3.4 (Pin_4), C2.1, D?.1 (K), R5.1, R6.1; no longer J3.1 (Pin_1)
- net BATT_SENSE: now also D?.2 (A)
- net ESP_TX: now also J3.1 (Pin_1); no longer J3.3 (Pin_3)
- net GND: now also J3.3 (Pin_3), C2.2, C4.2, C5.2, R11.2, SW1.1, SW2.2 (B); no longer J3.4 (Pin_4)
- net MOT_L_IN1: now also U1.4 (GPIO16); no longer U1.6 (GPIO12)
- net MOT_R_IN1: now also U1.13 (MOSI); no longer U1.17 (GPIO2)
- net MOT_R_IN2: now also U1.14 (SCLK); no longer U1.18 (GPIO0)
- net MOT_R_PWM: now also U1.6 (GPIO12); no longer U1.16 (GPIO15)
- net at R3.2, U1.3 (EN): now also C4.1, SW1.2
- new net: C5.1, R6.2, SW2.1 (A), U1.18 (GPIO0)
- new net: R11.1, U1.16 (GPIO15)
- new net: R5.2, U1.17 (GPIO2)
- no-connect marks 5 -> 2
Other:
- moved on the sheet: C1, C6, C7, C8, C9, J3, R10, R12, R3, R4, U2

Commit message: more pcb layout
Parts:
- removed J2: Conn_01x02, Connector_PinHeader_2.54mm:PinHeader_1x02_P2.54mm_Vertical, symbol Connector_Generic:Conn_01x02
- removed Q1, Q2: AO3401A, Package_TO_SOT_SMD:SOT-23, symbol Transistor_FET:AO3401A
- removed R1: 10k, Resistor_SMD:R_0805_2012Metric, symbol Device:R
- removed R8: 1k, Resistor_SMD:R_0805_2012Metric, symbol Device:R
- removed SW2: SW_SPST, symbol Switch:SW_SPST
- added Q1: QM6015D, Package_TO_SOT_SMD:TO-252-2, symbol Transistor_FET:QM6015D
- added SW1: SW_SPST, Connector_AMASS:AMASS_XT30U-F_1x02_P5.0mm_Vertical, symbol Switch:SW_SPST
- added SW3: SW_Push, Button_Switch_SMD:SW_Push_1P1T_NO_6x6mm_H9.5mm, symbol Switch:SW_Push
- C3: footprint Capacitor_THT:CP_Radial_D10.0mm_P5.00mm -> Capacitor_THT:CP_Radial_D10.0mm_P7.50mm
- D2: renamed from D?; footprint (none) -> Diode_SMD:D_0805_2012Metric
- SW2: renamed from SW1; footprint (none) -> Button_Switch_SMD:SW_Push_1P1T_NO_6x6mm_H9.5mm
- renumbered D2 to D3, D3 to D4, D4 to D5, D5 to D6, J3 to J2, J4 to J3, J5 to J4, J6 to J5, J7 to J6, R2 to R1, R12 to R10, R13 to R11, R14 to R12, R15 to R13, R16 to R14, R3 to R2, R4 to R3, R5 to R4, R6 to R5, R7 to R6, R9 to R7, R10 to R8, R11 to R9
Connections:
- net GND: now also SW3.2
- net V_INPUT: now also Q1.3 (S), SW1.2 (B)
- net V_POWER: now also Q1.2 (D)
- net at C4.1, R2.2, SW2.2: now also U1.1 (~{RST}); no longer U1.3 (EN)
- net at C5.1, R5.2, U1.18 (GPIO0): now also SW3.1
- net at J1.1 (Pin_1): now also SW1.1 (A)
- net at R3.2: now also U1.3 (EN); no longer U1.1 (~{RST})
- net at R1.2, R7.1: now also Q1.1 (G)
Other:
- moved on the sheet: R3
